File: mainboard.kicad_sch (KiCad schematic)
At the start: 87 parts

Commit message: Add hardware README and schematic documentation
Parts:
- ACC_FPC1: value AFC01-S22FCA-00 -> ACC Scanning FPC connector
- COL_FPC1: value ADC Column FPC 1 -> FSR ADC FPC connector 1
- COL_FPC2: value ADC Column FPC 2 -> FSR ADC FPC connector 2
- ROW_FPC1: value Scanning Row FPC 1 -> FSR Scanning FPC connector 1
- ROW_FPC2: value Scanning Row FPC 2 -> FSR Scanning FPC connector 2
Other:
- note added: "ACC SCANNING MUX"
- note added: "FSR-array ADCs"
- note added: "FSR-array Scanning MUX"
- note added: "Microcontroller unit chip (STM32G474CETx)"
- note added: "Mounting Hole"
- note removed: "ACC MUX and FPC"
- note removed: "ADCs"
- note removed: "Scanning mux"
- company: (none) -> YANNAS
- title: (none) -> E-SKIN Mainboard
